File: KB-Prototype.kicad_pcb (KiCad board)
At the start: 2 copper layers, 145.3 x 57.2 mm, 45 parts, among them J1 Conn_01x04, J2 Conn_01x04, J3 Conn_01x04, SW1 SW_Push, U1 ATmega32U4-AU, Y1 Resonator_Small

Commit message: traced right half, added mounting holes
Parts:
- removed D2, D3, D5, D6, D8, D9: BAT54C, Package_TO_SOT_SMD:SOT-23
- removed J1: Conn_01x04, random-keyboard-parts:JST-SR-4
- removed MX10, MX11, MX12, MX15, MX16, MX17, MX18, MX3, MX4, MX5, MX6, MX9: MX-NoLED, MX_Only:MXOnly-1U-NoLED
- removed R2, R3: 4.7k, Resistor_SMD:R_0805_2012Metric
- added H1: MountingHole, random-keyboard-parts:Generic-Mounthole, F.Cu at (26.9, 26.8)
- added H2: MountingHole, random-keyboard-parts:Generic-Mounthole, F.Cu at (26.8, 78.0)
- added H3: MountingHole, random-keyboard-parts:Generic-Mounthole, F.Cu at (89.9, 26.8)
- added H4: MountingHole, random-keyboard-parts:Generic-Mounthole, F.Cu at (89.8, 78.0)
- moved C2 76.2 mm to (69.8, 46.8)
- moved C3 76.2 mm to (85.7, 50.0)
- moved C4 76.2 mm to (81.8, 63.5)
- moved SW1 76.2 mm to (71.0, 72.6)
- moved C5 76.2 mm to (67.8, 60.2)
- moved J2 76.2 mm to (66.7, 27.8)
- moved J3 76.2 mm to (78.5, 27.8)
- moved R1 76.2 mm to (66.3, 46.8)
- moved R4 76.2 mm to (68.3, 38.1)
- moved Y1 76.2 mm to (76.6, 44.6)
- moved C1 76.2 mm to (67.5, 54.8)
- moved R5 76.2 mm to (65.1, 38.1)
- moved R6 76.2 mm to (85.9, 59.7)
- moved R7 76.2 mm to (78.6, 65.7)
- moved U1 76.2 mm to (77.0, 54.8)
Connections:
- R7 pad 1: +5V -> GND
- U1 pad 37: ROW2 -> Net-(U1-Pad37)
- U1 pad 38: COL5 -> Net-(U1-Pad38)
- U1 pad 39: COL4 -> Net-(U1-Pad39)
- U1 pad 40: COL3 -> Net-(U1-Pad40)
- U1 pad 41: COL2 -> ROW2
- U1 pad 8: COL1 -> COL0
- U1 pad 9: COL0 -> COL1
Routing:
- net COL2: track 124.5 -> 0.00 mm, vias 1 -> 0
- net COL3: track 106.7 -> 0.00 mm, vias 1 -> 0
- net COL4: track 89.0 -> 0.00 mm, vias 1 -> 0
- net ROW2: track 120.5 -> 40.4 mm
- net COL0: track 159.5 -> 82.8 mm
- net ROW0: track 109.1 -> 32.9 mm
- net ROW1: track 107.7 -> 31.5 mm
- net COL1: track 140.3 -> 64.3 mm
- net COL5: track 71.5 -> 0.00 mm, vias 1 -> 0
- net +5V: track 161.3 -> 123.2 mm, vias 12 -> 7
- net Net-(D8-Pad2): track 19.7 -> 0.00 mm
- net Net-(D5-Pad2): track 19.7 -> 0.00 mm
- net Net-(D2-Pad2): track 19.7 -> 0.00 mm
- net Net-(D9-Pad2): track 19.7 -> 0.00 mm
- net Net-(D6-Pad2): track 19.7 -> 0.00 mm
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Other:
- board size 145.3 x 57.2 mm -> 69.1 x 57.2 mm
- board text added: "KB-Prototype RIGHT"
- board text removed: "KB-Prototype LEFT"

Commit message: generated gerbers
Routing:
- added copper zone on B.Cu, net GND
Changed lines of the file:
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@@
     (solder_mask_min_width 0.25)
     (aux_axis_origin 0 0)
-    (visible_elements 7FFFFFFF)
+    (visible_elements 7FFFEFFF)
     (pcbplotparams
-      (layerselection 0x010fc_ffffffff)
-      (usegerberextensions false)
+      (layerselection 0x010f0_ffffffff)
+      (usegerberextensions true)
       (usegerberattributes false)
       (usegerberadvancedattributes false)
@@
       (plotinvisibletext false)
       (padsonsilk false)
-      (subtractmaskfromsilk false)
+      (subtractmaskfromsilk true)
       (outputformat 1)
       (mirror false)
-      (drillshape 1)
+      (drillshape 0)
       (scaleselection 1)
-      (outputdirectory ""))
+      (outputdirectory "Gerbers"))
   )
   (net 0 "")
@@
   (segment (start 29.5275 30.7975) (end 29.5275 49.8475) (width 0.25) (layer F.Cu) (net 17))
   (segment (start 29.5275 49.8475) (end 29.5275 59.7535) (width 0.25) (layer F.Cu) (net 17))
-  (via (at 60.593421 53.567952) (size 0.8) (drill 0.4) (layers F.Cu B.Cu) (net 18))
-  (segment (start 60.99342 53.167953) (end 61.005047 53.167953) (width 0.25) (layer F.Cu) (net 18))
-  (segment (start 60.593421 53.567952) (end 60.99342 53.167953) (width 0.25) (layer F.Cu) (net 18))
-  (via (at 64.342299 52.394051) (size 0.8) (drill 0.4) (layers F.Cu B.Cu) (net 18))
-  (segment (start 61.005047 53.167953) (end 61.778949 52.394051) (width 0.25) (layer F.Cu) (net 18))
-  (segment (start 61.778949 52.394051) (end 64.342299 52.394051) (width 0.25) (layer F.Cu) (net 18))
-  (segment (start 71.29375 52.36875) (end 64.342299 52.36875) (width 0.25) (layer B.Cu) (net 18))
-  (segment (start 48.5775 32.38849) (end 48.5775 49.8475) (width 0.25) (layer F.Cu) (net 18))
-  (segment (start 48.5775 30.7975) (end 48.5775 32.38849) (width 0.25) (layer F.Cu) (net 18))
-  (segment (start 48.5775 49.8475) (end 48.5775 51.43849) (width 0.25) (layer F.Cu) (net 18))
-  (segment (start 48.5775 60.5155) (end 48.5775 60.7325) (width 0.25) (layer F.Cu) (net 18))
-  (segment (start 48.5775 60.5155) (end 48.5775 68.8975) (width 0.25) (layer F.Cu) (net 18))
   (via (at 60.579 54.737) (size 0.8) (drill 0.4) (layers F.Cu B.Cu) (net 17))
   (segment (start 60.579 54.737) (end 60.978999 54.337001) (width 0.25) (layer F.Cu) (net 17))
@@
   (segment (start 29.5275 59.7535) (end 29.5275 60.3885) (width 0.25) (layer F.Cu) (net 17))
   (segment (start 29.5275 60.3885) (end 29.5275 68.8975) (width 0.25) (layer F.Cu) (net 17))
+  (via (at 60.593421 53.567952) (size 0.8) (drill 0.4) (layers F.Cu B.Cu) (net 18))
+  (segment (start 60.99342 53.167953) (end 61.005047 53.167953) (width 0.25) (layer F.Cu) (net 18))
+  (segment (start 60.593421 53.567952) (end 60.99342 53.167953) (width 0.25) (layer F.Cu) (net 18))
+  (via (at 64.342299 52.394051) (size 0.8) (drill 0.4) (layers F.Cu B.Cu) (net 18))
+  (segment (start 61.005047 53.167953) (end 61.778949 52.394051) (width 0.25) (layer F.Cu) (net 18))
+  (segment (start 61.778949 52.394051) (end 64.342299 52.394051) (width 0.25) (layer F.Cu) (net 18))
+  (segment (start 71.29375 52.36875) (end 64.342299 52.36875) (width 0.25) (layer B.Cu) (net 18))
+  (segment (start 48.5775 32.38849) (end 48.5775 49.8475) (width 0.25) (layer F.Cu) (net 18))
+  (segment (start 48.5775 30.7975) (end 48.5775 32.38849) (width 0.25) (layer F.Cu) (net 18))
+  (segment (start 48.5775 49.8475) (end 48.5775 51.43849) (width 0.25) (layer F.Cu) (net 18))
+  (segment (start 48.5775 60.5155) (end 48.5775 60.7325) (width 0.25) (layer F.Cu) (net 18))
+  (segment (start 48.5775 60.5155) (end 48.5775 68.8975) (width 0.25) (layer F.Cu) (net 18))
   (via (at 48.5775 59.66875) (size 0.8) (drill 0.4) (layers F.Cu B.Cu) (net 18))
   (segment (start 48.5775 59.3725) (end 48.5775 59.66875) (width 0.25) (layer F.Cu) (net 18))
@@
   (segment (start 75.401 45.847) (end 75.381 45.827) (width 0.25) (layer B.Cu) (net 37))
   (segment (start 75.438 45.847) (end 75.401 45.847) (width 0.25) (layer B.Cu) (net 37))
+  (zone (net 1) (net_name GND) (layer B.Cu) (hatch edge 0.508)
+    (connect_pads (clearance 0.508))
+    (min_thickness 0.254)
+    (fill yes (arc_segments 32) (thermal_gap 0.508) (thermal_bridge_width 0.508) (smoothing fillet) (radius 0.5))
+    (polygon
+      (pts
+        (xy 71.755 49.53) (xy 71.755 60.071) (xy 82.296 60.071) (xy 82.296 49.53)
+      )
+    )
+  )
 )
